File: KiCad/geiger_entropy.kicad_pcb (KiCad board)
At the start: 2 copper layers, 53 x 63 mm, 37 parts, among them J1 AudioJack2, J2 USB_C_Receptacle_PowerOnly_6P, J3 ICSP, SW1 REV, SW2 FWD, SW3 RESET, U1 LM393, U2 ER_OLEDM0.91_1x-I2C, U3 ATmega328P-A, Y1 16MHz

Commit message: Update PCB to include M2.5 mounting holes
Parts:
- added REF**: MountingHole_2.7mm_M2.5_DIN965_Pad, MountingHole:MountingHole_2.7mm_M2.5_DIN965_Pad, F.Cu at (129.0, 96.0)
- added REF**: MountingHole_2.7mm_M2.5_DIN965_Pad, MountingHole:MountingHole_2.7mm_M2.5_DIN965_Pad, F.Cu at (167.0, 84.0)
- added REF**: MountingHole_2.7mm_M2.5_DIN965_Pad, MountingHole:MountingHole_2.7mm_M2.5_DIN965_Pad, F.Cu at (148.0, 75.0)
- added REF**: MountingHole_2.7mm_M2.5_DIN965_Pad, MountingHole:MountingHole_2.7mm_M2.5_DIN965_Pad, F.Cu at (166.0, 122.0)
- added REF**: MountingHole_2.7mm_M2.5_DIN965_Pad, MountingHole:MountingHole_2.7mm_M2.5_DIN965_Pad, F.Cu at (129.0, 122.0)
- R10: value 1k -> 2.2k
- moved REF** 10.0 mm to (129.0, 107.0)
- moved G*** 5.00 mm to (172.0, 89.0), turned to 90 degrees
- moved SW1 5.00 mm to (141.0, 124.5)
- moved SW2 5.00 mm to (161.0, 124.5)
Routing:
- net /D5: track 33.2 -> 31.8 mm
- net /D11/MOSI: track 44.3 -> 43.0 mm
- net /D4: track 32.4 -> 33.0 mm
Other:
- board text added: "///// CAUTION /////////////////////////////// OPERATION MAY CREATE PARALLEL UNIVERSES ////"
- board text added: "https://github.com/captainchapster/Entropy32-Plus"
- board text removed: "///// CAUTION ///////////////////////// OPERATION MAY CREATE PARALLEL UNIVERSES"
- board text removed: "NC"

Commit message: Remove PCB mounting holes, satisfied with existing enclosure design
Parts:
- removed the REF** at (129.0, 96.0)
- removed the REF** at (167.0, 84.0)
- removed the REF** at (148.0, 75.0)
- removed the REF** at (166.0, 122.0)
- removed the REF** at (129.0, 122.0)
- moved REF** 10.0 mm to (129.0, 97.0)
- moved G*** 5.00 mm to (169.0, 85.0), turned to 180 degrees
- moved SW1 5.00 mm to (136.0, 124.5)
- moved SW2 5.00 mm to (166.0, 124.5)
Routing:
- net /D5: track 31.8 -> 33.1 mm
- net /D4: track 33.0 -> 32.4 mm
- net GND: vias 112 -> 121

Commit message: Update PCB
Routing:
- net GND: vias 121 -> 122
Changed lines of the file:
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@@
+	)
+	(via
+		(at 133 111)
+		(size 0.6)
+		(drill 0.3)
+		(layers "F.Cu" "B.Cu")
+		(free yes)
+		(net "GND")
 	)
 	(via

Commit message: Update PCB with more vias and a missing ISP program header annotation
Routing:
- net GND: vias 122 -> 131
Other:
- board text added: "NC"
Changed lines of the file:
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@@
+		)
+	)
+	(gr_text "NC"
+		(at 150 73 45)
+		(layer "F.SilkS")
+		(effects
+			(font
+				(face "Unispace")
+				(size 0.5 0.5)
+				(thickness 0.125)
+				(bold yes)
+			)
+			(justify right)
+		)
+		(render_cache "NC" 45
+			(polygon
+				(pts
+					(xy 149.241013 73.25311) (xy 149.662458 73.433156) (xy 149.361712 73.13241) (xy 149.422051 73.072071)
+					(xy 149.821714 73.471734) (xy 149.735167 73.558281) (xy 149.356272 73.401011) (xy 149.624355 73.669094)
+					(xy 149.564512 73.728936) (xy 149.164849 73.329273)
+				)
+			)
+			(polygon
+				(pts
+					(xy 149.714399 72.779724) (xy 149.764354 72.829679) (xy 149.63625 72.957783) (xy 149.62954 72.966988)
+					(xy 149.626341 72.97758) (xy 149.62609 72.989087) (xy 149.628348 73.001823) (xy 149.632912 73.014533)
+					(xy 149.6402 73.028053) (xy 149.660493 73.053268) (xy 149.842007 73.234782) (xy 149.866488 73.254341)
+					(xy 149.892459 73.266452) (xy 149.905222 73.26899) (xy 149.916961 73.268675) (xy 149.92776 73.265284)
+					(xy 149.936995 73.258529) (xy 150.0651 73.130424) (xy 150.114062 73.179386) (xy 149.952819 73.340629)
+					(xy 149.934108 73.355073) (xy 149.913248 73.363404) (xy 149.890674 73.366293) (xy 149.866488 73.364138)
+					(xy 149.842293 73.357204) (xy 149.816792 73.345098) (xy 149.79248 73.328877) (xy 149.768801 73.307987)
+					(xy 149.587288 73.126474) (xy 149.565936 73.102326) (xy 149.549444 73.077749) (xy 149.537155 73.051946)
+					(xy 149.530165 73.027297) (xy 149.528001 73.002683) (xy 149.530899 72.980062) (xy 149.539134 72.959237)
+					(xy 149.553157 72.940966)
+				)
+			)
 		)
 	)
@@
 	)
 	(via
+		(at 146 77)
+		(size 0.6)
+		(drill 0.3)
+		(layers "F.Cu" "B.Cu")
+		(free yes)
+		(net "GND")
+	)
+	(via
+		(at 136 94)
+		(size 0.6)
+		(drill 0.3)
+		(layers "F.Cu" "B.Cu")
+		(free yes)
+		(net "GND")
+	)
+	(via
 		(at 125 126)
 		(size 0.6)
@@
 	)
 	(via
+		(at 146 71)
+		(size 0.6)
+		(drill 0.3)
+		(layers "F.Cu" "B.Cu")
+		(free yes)
+		(net "GND")
+	)
+	(via
 		(at 146 116)
 		(size 0.6)
@@
 	)
 	(via
+		(at 150 77)
+		(size 0.6)
+		(drill 0.3)
+		(layers "F.Cu" "B.Cu")
+		(free yes)
+		(net "GND")
+	)
+	(via
 		(at 129 82)
 		(size 0.6)
@@
 	)
 	(via
-		(at 162 93)
+		(at 162 94)
 		(size 0.6)
 		(drill 0.3)
@@
 	)
 	(via
-		(at 159 93)
+		(at 159 94)
 		(size 0.6)
 		(drill 0.3)
@@
 	)
 	(via
+		(at 150 74)
+		(size 0.6)
+		(drill 0.3)
+		(layers "F.Cu" "B.Cu")
+		(free yes)
+		(net "GND")
+	)
+	(via
 		(at 148 116)
 		(size 0.6)
@@
 	)
 	(via
+		(at 153 94)
+		(size 0.6)
+		(drill 0.3)
+		(layers "F.Cu" "B.Cu")
+		(free yes)
+		(net "GND")
+	)
+	(via
 		(at 170 95)
 		(size 0.6)
@@
 	)
 	(via
+		(at 156 94)
+		(size 0.6)
+		(drill 0.3)
+		(layers "F.Cu" "B.Cu")
+		(free yes)
+		(net "GND")
+	)
+	(via
 		(at 160 74)
 		(size 0.6)
@@
 	)
 	(via
+		(at 139 94)
+		(size 0.6)
+		(drill 0.3)
+		(layers "F.Cu" "B.Cu")
+		(free yes)
+		(net "GND")
+	)
+	(via
 		(at 136 99)
 		(size 0.6)
@@
 		(size 0.6)
 		(drill 0.3)
+		(layers "F.Cu" "B.Cu")
+		(free yes)
+		(net "GND")
+	)
+	(via
+		(at 146 74)
+		(size 0.6)
+		(drill 0.3)
