File: KiCad/geiger_entropy.kicad_sch (KiCad schematic)
At the start: 34 parts, among them J1 AudioJack2, J2 USB_C_Receptacle_PowerOnly_6P, J3 ICSP, SW1 REV, SW2 FWD, SW3 RESET, U1 LM393, U2 ER_OLEDM0.91_1x-I2C, U3 ATmega328P-A, Y1 16MHz

Commit message: Update firmware and increase green LED resistor to 2.2k from 1k.
Parts:
- R10: value 1k -> 2.2k
Changed lines of the file:
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@@
 			)
 		)
-		(property "Value" "1k"
+		(property "Value" "2.2k"
 			(at 215.9 106.6799 0)
 			(show_name no)

Commit message: Update schematics
Other:
- note added: "1"
- note added: "16/09/2026"
- note added: "Entropy32 Plus"
- note added: "Entropy32 Plus, the universe bifurcator - by Alexander Higgins"
Changed lines of the file:
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@@
 	(generator_version "10.0")
 	(paper "A4")
+	(text "Entropy32 Plus, the universe bifurcator - by Alexander Higgins"
+		(exclude_from_sim no)
+		(at 188.722 189.992 0)
+		(effects
+			(font
+				(size 1.27 1.27)
+			)
+			(justify left)
+		)
+	)
+	(text "1"
+		(exclude_from_sim no)
+		(at 270.51 193.548 0)
+		(effects
+			(font
+				(size 1.27 1.27)
+			)
+		)
+	)
+	(text "Entropy32 Plus"
+		(exclude_from_sim no)
+		(at 179.324 174.244 0)
+		(effects
+			(font
+				(size 6.35 6.35)
+				(thickness 1.27)
+				(bold yes)
+				(italic yes)
+			)
+			(justify left)
+		)
+	)
+	(text "16/09/2026"
+		(exclude_from_sim no)
+		(at 214.122 193.548 0)
+		(effects
+			(font
+				(size 1.27 1.27)
+			)
+		)
+	)
 	(junction
 		(at 88.9 144.78)
